File: redwood.sch (KiCad schematic (older format))
At the start: 35 parts, among them J1 Haptic, J2 TRRS, K1 diode-choc, K10 diode-choc, K11 diode-choc, K12 diode-choc, K13 diode-choc, K14 diode-choc, K15 diode-choc, K16 diode-choc, K17 diode-choc, K18 diode-choc, K19 diode-choc, K2 diode-choc, K20 diode-choc, K21 diode-choc, K22 diode-choc, K23 diode-choc, K24 diode-choc, K3 diode-choc, K4 diode-choc, K5 diode-choc, K6 diode-choc, K7 diode-choc, K8 diode-choc, K9 diode-choc, SW1 Reset, U1 ProMicro_r

Commit message: Rename project to Redwood from LongFir
Parts:
- D1, D2, D3, D4, D5: footprint longfir:SK6812-MINI-E -> redwood:SK6812-MINI-E; symbol longfir:SK6812-MINI-E -> redwood:SK6812-MINI-E
- J1: footprint longfir:PomoroniHaptic -> redwood:PomoroniHaptic
- J2: footprint longfir:MJ-4PP-9 -> redwood:MJ-4PP-9; symbol longfir:TRRS -> redwood:TRRS
- K1, K10, K11, K12, K13, K14, K15, K16, K17, K18, K19, K2, K20, K21, K22, K23, K24, K3, K4, K5, K6, K7, K8, K9: footprint longfir:pg1350-DR -> redwood:pg1350-DR; symbol longfir:diode-choc -> redwood:diode-choc
- R1, R2: footprint longfir:R_0805_2012Metric_DoubleSided -> redwood:R_0805_2012Metric_DoubleSided
- SW1: footprint longfir:SW_Tactile_SPST_Angled_MJTP1117 -> redwood:SW_Tactile_SPST_Angled_MJTP1117
- U1: footprint longfir:ProMicro_v2 -> redwood:ProMicro_v2

Commit message: Scheme: encoder, symbols for hardware bits
Parts:
- removed K20: diode-choc, redwood:pg1350-DR, symbol redwood:diode-choc
- added D6: Diode, redwood:D_SOD-123_rev, symbol ki_device:D_Small
- added H1: Tenting_Mount, redwood:Tenting_Puck, symbol redwood:Tenting_Mounts
- added H2: Trackball, redwood:Pimoroni_Trackball, symbol redwood:Trackball_Mounts
- added K20: choc_rotary, redwood:pg1350-DR_rotary, symbol redwood:choc_rotary
- added V1: Via, mmccoyd:VIA-0.8mm, symbol redwood:Via
- J1: footprint redwood:PomoroniHaptic -> redwood:Pimoroni_Haptic
- R1: value R:SCL -> R:I2C; footprint redwood:R_0805_2012Metric_DoubleSided -> redwood:R_0805_2012Metric
- R2: value R:SDA -> R:I2C; footprint redwood:R_0805_2012Metric_DoubleSided -> redwood:R_0805_2012Metric
Connections:
- net GND: now also K20.C, V1.1 (via)
- net col0: now also K20.S1
- net row3: now also D6.1 (K)
- net enc_a: now reaches U1.19 (A2/F5)
- net enc_a: now also K20.A
- net enc_b: now reaches U1.20 (A3/F4)
- net enc_b: now also K20.B
- new net: D6.2 (A), K20.S2
- no-connect marks 6 -> 4
Other:
- moved on the sheet: D1, D2, D3, D4, D5, J1, J2, R1, R2, SW1, U1
