File: redwood.kicad_pcb (KiCad board)
At the start: 2 copper layers, 136.6 x 97.9 mm, 36 parts, among them J1 Haptic, J2 TRRS, K1 diode-choc, K10 diode-choc, K11 diode-choc, K12 diode-choc, K13 diode-choc, K14 diode-choc, K15 diode-choc, K16 diode-choc, K17 diode-choc, K18 diode-choc, K19 diode-choc, K2 diode-choc, K20 diode-choc, K21 diode-choc, K22 diode-choc, K23 diode-choc, K24 diode-choc, K3 diode-choc, K4 diode-choc, K5 diode-choc, K6 diode-choc, K7 diode-choc, K8 diode-choc, K9 diode-choc, SW1 Reset, U1 ProMicro_r

Commit message: Rename project to Redwood from LongFir
Parts:
- D1, D2, D3, D4, D5: footprint longfir:SK6812-MINI-E -> redwood:SK6812-MINI-E
- J1: footprint longfir:PomoroniHaptic -> redwood:PomoroniHaptic
- J2: footprint longfir:MJ-4PP-9 -> redwood:MJ-4PP-9
- K1, K10, K11, K12, K13, K14, K15, K16, K17, K18, K19, K2, K20, K21, K22, K23, K24, K3, K4, K5, K6, K7, K8, K9: footprint longfir:pg1350-DR -> redwood:pg1350-DR
- R1, R2: footprint longfir:R_0805_2012Metric_DoubleSided -> redwood:R_0805_2012Metric_DoubleSided
- REF**: footprint longfir:Tenting_Puck -> redwood:Tenting_Puck
- SW1: footprint longfir:SW_Tactile_SPST_Angled_MJTP1117 -> redwood:SW_Tactile_SPST_Angled_MJTP1117
- U1: footprint longfir:ProMicro_v2 -> redwood:ProMicro_v2
Changed lines of the file:
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@@
     (add_net VCC)
   )
-  (module longfir:SW_Tactile_SPST_Angled_MJTP1117 (layer F.Cu)
+  (module redwood:SW_Tactile_SPST_Angled_MJTP1117 (layer F.Cu)
     (at 221.28 111.98 285)
     (descr "tactile switch SPST right angle, PTS645VL39-2 LFS")
@@
     )
   )
-  (module longfir:pg1350-DR (layer F.Cu)
+  (module redwood:pg1350-DR (layer F.Cu)
     (at 218.322328 141.509268 135)
     (fp_text reference K24 (at 0 0 135) (layer F.Fab) hide
@@
     (pad "" np_thru_hole circle (at 0 -4.5 135) (size 3.4 3.4) (drill 3.4) (layers *.Cu *.Mask))
   )
-  (module longfir:pg1350-DR (layer F.Cu)
+  (module redwood:pg1350-DR (layer F.Cu)
     (at 201.728276 128.652806 150)
     (fp_text reference K23 (at 0 0 150) (layer F.Fab) hide
@@
     (pad "" np_thru_hole circle (at 0 -4.5 150) (size 3.4 3.4) (drill 3.4) (layers *.Cu *.Mask))
   )
-  (module longfir:pg1350-DR (layer F.Cu)
+  (module redwood:pg1350-DR (layer F.Cu)
     (at 182.274686 120.54 165)
     (fp_text reference K22 (at 0 0 165) (layer F.Fab) hide
@@
     (pad "" np_thru_hole circle (at 0 -4.5 165) (size 3.4 3.4) (drill 3.4) (layers *.Cu *.Mask))
   )
-  (module longfir:pg1350-DR (layer F.Cu)
+  (module redwood:pg1350-DR (layer F.Cu)
     (at 161.5 117.5 180)
     (fp_text reference K21 (at 0 0) (layer F.Fab) hide
@@
     (pad "" np_thru_hole circle (at 0 -4.5 180) (size 3.4 3.4) (drill 3.4) (layers *.Cu *.Mask))
   )
-  (module longfir:pg1350-DR locked (layer F.Cu)
+  (module redwood:pg1350-DR locked (layer F.Cu)
     (at 136 119 180)
     (fp_text reference K20 (at 0 0) (layer F.Fab) hide
@@
     (pad "" np_thru_hole circle (at 0 -4.5 180) (size 3.4 3.4) (drill 3.4) (layers *.Cu *.Mask))
   )
-  (module longfir:pg1350-DR (layer F.Cu)
+  (module redwood:pg1350-DR (layer F.Cu)
     (at 210.228276 113.930374 150)
     (fp_text reference K19 (at 0 0 150) (layer F.Fab) hide
@@
     (pad "" np_thru_hole circle (at 0 -4.5 150) (size 3.4 3.4) (drill 3.4) (layers *.Cu *.Mask))
   )
-  (module longfir:pg1350-DR locked (layer F.Cu)
+  (module redwood:pg1350-DR locked (layer F.Cu)
     (at 190 103 180)
     (fp_text reference K18 (at 0 0) (layer F.Fab) hide
@@
     (pad "" np_thru_hole circle (at 0 -4.5 180) (size 3.4 3.4) (drill 3.4) (layers *.Cu *.Mask))
   )
-  (module longfir:pg1350-DR locked (layer F.Cu)
+  (module redwood:pg1350-DR locked (layer F.Cu)
     (at 172 100.5 180)
     (fp_text reference K17 (at 0 0) (layer F.Fab) hide
@@
     (pad "" np_thru_hole circle (at 0 -4.5 180) (size 3.4 3.4) (drill 3.4) (layers *.Cu *.Mask))
   )
-  (module longfir:pg1350-DR locked (layer F.Cu)
+  (module redwood:pg1350-DR locked (layer F.Cu)
     (at 154 95 180)
     (fp_text reference K16 (at 0 0) (layer F.Fab) hide
@@
     (pad "" np_thru_hole circle (at 0 -4.5 180) (size 3.4 3.4) (drill 3.4) (layers *.Cu *.Mask))
   )
-  (module longfir:pg1350-DR locked (layer F.Cu)
+  (module redwood:pg1350-DR locked (layer F.Cu)
     (at 136 102 180)
     (fp_text reference K15 (at 0 0) (layer F.Fab) hide
@@
     (pad "" np_thru_hole circle (at 0 -4.5 180) (size 3.4 3.4) (drill 3.4) (layers *.Cu *.Mask))
   )
-  (module longfir:pg1350-DR locked (layer F.Cu)
+  (module redwood:pg1350-DR locked (layer F.Cu)
     (at 118 114 180)
     (fp_text reference K14 (at 0 0) (layer F.Fab) hide
@@
     (pad "" np_thru_hole circle (at 0 -4.5 180) (size 3.4 3.4) (drill 3.4) (layers *.Cu *.Mask))
   )
-  (module longfir:pg1350-DR locked (layer F.Cu)
+  (module redwood:pg1350-DR locked (layer F.Cu)
     (at 100 114 180)
     (fp_text reference K13 (at 0 0) (layer F.Fab) hide
@@
     (pad "" np_thru_hole circle (at 0 -4.5 180) (size 3.4 3.4) (drill 3.4) (layers *.Cu *.Mask))
   )
-  (module longfir:pg1350-DR locked (layer F.Cu)
+  (module redwood:pg1350-DR locked (layer F.Cu)
     (at 190 86 180)
     (fp_text reference K12 (at 0 0) (layer F.Fab) hide
@@
     (pad "" np_thru_hole circle (at 0 -4.5 180) (size 3.4 3.4) (drill 3.4) (layers *.Cu *.Mask))
   )
-  (module longfir:pg1350-DR locked (layer F.Cu)
+  (module redwood:pg1350-DR locked (layer F.Cu)
     (at 172 83.5 180)
     (fp_text reference K11 (at 0 0) (layer F.Fab) hide
@@
     (pad "" np_thru_hole circle (at 0 -4.5 180) (size 3.4 3.4) (drill 3.4) (layers *.Cu *.Mask))
   )
-  (module longfir:pg1350-DR locked (layer F.Cu)
+  (module redwood:pg1350-DR locked (layer F.Cu)
     (at 154 78 180)
     (fp_text reference K10 (at 0 0) (layer F.Fab) hide
@@
     (pad "" np_thru_hole circle (at 0 -4.5 180) (size 3.4 3.4) (drill 3.4) (layers *.Cu *.Mask))
   )
-  (module longfir:pg1350-DR locked (layer F.Cu)
+  (module redwood:pg1350-DR locked (layer F.Cu)
     (at 136 85 180)
     (fp_text reference K9 (at 0 0) (layer F.Fab) hide
@@
     (pad "" np_thru_hole circle (at 0 -4.5 180) (size 3.4 3.4) (drill 3.4) (layers *.Cu *.Mask))
   )
-  (module longfir:pg1350-DR locked (layer F.Cu)
+  (module redwood:pg1350-DR locked (layer F.Cu)
     (at 118 97 180)
     (fp_text reference K8 (at 0 0) (layer F.Fab) hide
@@
     (pad "" np_thru_hole circle (at 0 -4.5 180) (size 3.4 3.4) (drill 3.4) (layers *.Cu *.Mask))
   )
-  (module longfir:pg1350-DR locked (layer F.Cu)
+  (module redwood:pg1350-DR locked (layer F.Cu)
     (at 100 97 180)
     (fp_text reference K7 (at 0 0) (layer F.Fab) hide
@@
     (pad "" np_thru_hole circle (at 0 -4.5 180) (size 3.4 3.4) (drill 3.4) (layers *.Cu *.Mask))
   )
-  (module longfir:pg1350-DR locked (layer F.Cu)
+  (module redwood:pg1350-DR locked (layer F.Cu)
     (at 190 69 180)
     (fp_text reference K6 (at 0 0) (layer F.Fab) hide
@@
     (pad "" np_thru_hole circle (at 0 -4.5 180) (size 3.4 3.4) (drill 3.4) (layers *.Cu *.Mask))
   )
-  (module longfir:pg1350-DR locked (layer F.Cu)
+  (module redwood:pg1350-DR locked (layer F.Cu)
     (at 172 66.5 180)
     (fp_text reference K5 (at 0 0) (layer F.Fab) hide
@@
     (pad "" np_thru_hole circle (at 0 -4.5 180) (size 3.4 3.4) (drill 3.4) (layers *.Cu *.Mask))
   )
-  (module longfir:pg1350-DR locked (layer F.Cu)
+  (module redwood:pg1350-DR locked (layer F.Cu)
     (at 154 61 180)
     (fp_text reference K4 (at 0 0) (layer F.Fab) hide
@@
     (pad "" np_thru_hole circle (at 0 -4.5 180) (size 3.4 3.4) (drill 3.4) (layers *.Cu *.Mask))
   )
-  (module longfir:pg1350-DR locked (layer F.Cu)
+  (module redwood:pg1350-DR locked (layer F.Cu)
     (at 136 68 180)
     (fp_text reference K3 (at 0 0) (layer F.Fab) hide
@@
     (pad "" np_thru_hole circle (at 0 -4.5 180) (size 3.4 3.4) (drill 3.4) (layers *.Cu *.Mask))
   )
-  (module longfir:pg1350-DR locked (layer F.Cu)
+  (module redwood:pg1350-DR locked (layer F.Cu)
     (at 118 80 180)
     (fp_text reference K2 (at 0 0) (layer F.Fab) hide
@@
     (pad "" np_thru_hole circle (at 0 -4.5 180) (size 3.4 3.4) (drill 3.4) (layers *.Cu *.Mask))
   )
-  (module longfir:pg1350-DR locked (layer F.Cu)
+  (module redwood:pg1350-DR locked (layer F.Cu)
     (at 100 80 180)
     (fp_text reference K1 (at 0 0) (layer F.Fab) hide
@@
     (pad "" np_thru_hole circle (at 0 -4.5 180) (size 3.4 3.4) (drill 3.4) (layers *.Cu *.Mask))
   )
-  (module longfir:PomoroniHaptic (layer F.Cu)
+  (module redwood:PomoroniHaptic (layer F.Cu)
     (at 214.975 93.45)
     (descr "Through hole header 2.54mm pitch and one of two mount points for Pomoroni Haptic PIM452")
@@
       (net 11 GND))
   )
-  (module longfir:R_0805_2012Metric_DoubleSided (layer F.Cu)
+  (module redwood:R_0805_2012Metric_DoubleSided (layer F.Cu)
     (at 206.025 103.89 90)
     (descr "Resistor SMD 0805 (2012 Metric), square (rectangular) end terminal, IPC_7351 nominal, (Body size source: IPC-SM-782 page 72, https://www.pcb-3d.com/wordpress/wp-content/uploads/ipc-sm-782a_amendment_1_and_2.pdf), generated with kicad-footprint-generator")
@@
     )
   )
-  (module longfir:R_0805_2012Metric_DoubleSided (layer F.Cu)
+  (module redwood:R_0805_2012Metric_DoubleSided (layer F.Cu)
     (at 204 103.89 90)
     (descr "Resistor SMD 0805 (2012 Metric), square (rectangular) end terminal, IPC_7351 nominal, (Body size source: IPC-SM-782 page 72, https://www.pcb-3d.com/wordpress/wp-content/uploads/ipc-sm-782a_amendment_1_and_2.pdf), generated with kicad-footprint-generator")
@@
     )
   )
-  (module longfir:ProMicro_v2 (layer F.Cu)
+  (module redwood:ProMicro_v2 (layer F.Cu)
     (at 210 86.63)
     (fp_text reference U1 (at -1.27 2.762 270) (layer F.SilkS) hide
@@
       (net 21 "Net-(U1-Pad24)"))
   )
-  (module longfir:MJ-4PP-9 (layer F.Cu)
+  (module redwood:MJ-4PP-9 (layer F.Cu)
     (at 214.98 129.36 90)
     (fp_text reference J2 (at -1.99 10.82 270) (layer F.Fab)
@@
     )
   )
-  (module longfir:SK6812-MINI-E (layer F.Cu)
+  (module redwood:SK6812-MINI-E (layer F.Cu)
     (at 131.73 115.11)
     (fp_text reference D5 (at 0 -2.2 unlocked) (layer F.Fab)
@@
     )
   )
-  (module longfir:SK6812-MINI-E (layer F.Cu)
+  (module redwood:SK6812-MINI-E (layer F.Cu)
     (at 161.486067 113.577196)
     (fp_text reference D4 (at 0 -2.2 unlocked) (layer F.Fab)
@@
     )
   )
-  (module longfir:SK6812-MINI-E (layer F.Cu)
+  (module redwood:SK6812-MINI-E (layer F.Cu)
     (at 183.313671 116.792767 345)
     (fp_text reference D3 (at 0 -2.2 345 unlocked) (layer F.Fab)
@@
     )
   )
-  (module longfir:SK6812-MINI-E (layer F.Cu)
+  (module redwood:SK6812-MINI-E (layer F.Cu)
     (at 203.699418 125.287879 330)
     (fp_text reference D2 (at 0 -2.2 330 unlocked) (layer F.Fab)
@@
     )
   )
-  (module longfir:SK6812-MINI-E (layer F.Cu)
+  (module redwood:SK6812-MINI-E (layer F.Cu)
     (at 208.481456 108.542398 330)
     (fp_text reference D1 (at 0 -2.2 330 unlocked) (layer F.Fab)
@@
     )
   )
-  (module longfir:Tenting_Puck (layer F.Cu)
+  (module redwood:Tenting_Puck (layer F.Cu)
     (at 163.01 81.96)
     (fp_text reference REF** (at 7.6835 1.4605) (layer F.Fab)

Commit message: PCB: Rotary encoder
Parts:
- removed REF**: Tenting Puck, redwood:Tenting_Puck
- added D6: Diode, redwood:D_SOD-123_rev, F.Cu at (140.9, 115.0)
- added H1: Tenting_Mount, redwood:Tenting_Puck, F.Cu at (163.0, 82.0)
- added H2: Trackball, redwood:Pimoroni_Trackball, F.Cu at (212.0, 112.9)
- added V1: Via, mmccoyd:VIA-0.8mm, F.Cu at (121.0, 123.9)
- J1: footprint redwood:PomoroniHaptic -> redwood:Pimoroni_Haptic
- K20: value diode-choc -> choc_rotary; footprint redwood:pg1350-DR -> redwood:pg1350-DR_rotary
- R1: value R:SCL -> R:I2C; footprint redwood:R_0805_2012Metric_DoubleSided -> redwood:R_0805_2012Metric
- R2: value R:SDA -> R:I2C; footprint redwood:R_0805_2012Metric_DoubleSided -> redwood:R_0805_2012Metric
- moved R2 28.0 mm to (220.6, 80.0), turned to 270 degrees
- moved R1 21.4 mm to (220.6, 90.4)
- moved SW1 2.51 mm to (221.1, 109.5)
- moved D1 0.14 mm to (208.5, 108.4)
Connections:
- U1 pad 19: Net-(U1-Pad19) -> enc_a
- U1 pad 20: Net-(U1-Pad20) -> enc_b
Routing:
- net enc_a: track 0.00 -> 125.8 mm, vias 0 -> 2
- net enc_b: track 0.00 -> 121.0 mm, vias 0 -> 2
- net VCC: track 197.4 -> 224.7 mm, vias 9 -> 10
- net col0: track 222.3 -> 202.8 mm, vias 7 -> 6
- net Net-(U1-Pad20): track 14.4 -> 0.00 mm, vias 1 -> 0
- net Net-(U1-Pad19): track 14.4 -> 0.00 mm, vias 1 -> 0
- net Net-(D6-Pad2): track 0.00 -> 13.5 mm
- net col1: track 208.9 -> 196.3 mm
- net SCL: track 49.3 -> 41.6 mm
- net SDA: track 46.4 -> 42.3 mm
- net row3: track 159.8 -> 156.1 mm, vias 4 -> 6
- net reset: track 55.5 -> 52.2 mm
- net row2: track 137.8 -> 136.0 mm
- net col2: track 177.5 -> 178.9 mm
- net data: track 78.8 -> 77.8 mm
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