File: kicad/hillside.sch (KiCad schematic (older format))
At the start: 80 parts, among them J1 Haptic, J2 TRRS, J3 Batt_Pos, J4 Batt_GND, K1 SW_Key, K10 SW_Key, K11 SW_Key, K12 SW_Key, K13 SW_Key, K14 SW_Key, K15 SW_Key, K16 SW_Key, K17 SW_Key, K18 SW_Key, K19 SW_Key, K2 SW_Key, K20 SW_Rotary, K21 SW_Key, K22 SW_Key, K23 SW_Key, K24 SW_Key, K3 SW_Key, K4 SW_Key, K5 SW_Key, K6 SW_Key, K7 SW_Key, K8 SW_Key, K9 SW_Key, SW1 Reset, SW2 SW_Power, U1 ProMicro_r

Commit message: Rename to Hillside
Parts:
- H1: footprint redwood:Tenting_Puck -> hillside:Tenting_Puck; symbol redwood:Mount_Tenting -> hillside:Mount_Tenting
- H2: footprint redwood:Pimoroni_Trackball -> hillside:Pimoroni_Trackball; symbol redwood:Mount_Trackball -> hillside:Mount_Trackball
- H3: footprint redwood:Hillside_Scene -> hillside:Hillside_Scene; symbol redwood:Scene -> hillside:Scene
- J1: footprint redwood:Pimoroni_Haptic -> hillside:Pimoroni_Haptic
- J2: footprint redwood:MJ-4PP-9 -> hillside:MJ-4PP-9; symbol redwood:TRRS -> hillside:TRRS
- K1, K10, K11, K12, K13, K14, K15, K16, K17, K18, K19, K2, K21, K22, K23, K24, K3, K4, K5, K6, K7, K8, K9: footprint redwood:pg1350-R -> hillside:pg1350-R; symbol redwood:SW_Key -> hillside:SW_Key
- K20: footprint redwood:pg1350-DR_rotary -> hillside:pg1350-DR_rotary; symbol redwood:SW_Rotary -> hillside:SW_Rotary
- SW1: symbol redwood:SW_PUSH -> hillside:SW_PUSH
- U1: footprint redwood:ProMicro_v2 -> hillside:ProMicro_v2; symbol redwood:ProMicro_r -> hillside:ProMicro_r
Changed lines of the file:
@@
 reset
 $Comp
-L redwood:ProMicro_r U1
+L hillside:ProMicro_r U1
 U 1 1 6162C399
 P 3000 5400
 F 0 "U1" H 3050 6387 60  0000 C CNN
 F 1 "ProMicro_r" H 3050 6281 60  0000 C CNN
-F 2 "redwood:ProMicro_v2" H 3150 4350 60  0001 C CNN
+F 2 "hillside:ProMicro_v2" H 3150 4350 60  0001 C CNN
 F 3 "" H 3150 4350 60  0000 C CNN
 	1    3000 5400
@@
 F 0 "J1" H 8700 4950 50  0000 L CNN
 F 1 "Haptic" H 8700 4850 50  0000 L CNN
-F 2 "redwood:Pimoroni_Haptic" H 8600 4900 50  0001 C CNN
+F 2 "hillside:Pimoroni_Haptic" H 8600 4900 50  0001 C CNN
 F 3 "" H 8600 4900 50  0001 C CNN
 	1    8600 4900
@@
 	8300 4700 8400 4700
 $Comp
-L redwood:TRRS J2
+L hillside:TRRS J2
 U 1 1 61A70C2C
 P 2900 6800
 F 0 "J2" H 3450 6800 50  0000 L CNN
 F 1 "TRRS" H 3450 6700 50  0000 L CNN
-F 2 "redwood:MJ-4PP-9" V 4050 6650 50  0001 C CNN
+F 2 "hillside:MJ-4PP-9" V 4050 6650 50  0001 C CNN
 F 3 "~" V 4050 6650 50  0001 C CNN
 	1    2900 6800
@@
 Connection ~ 2800 7000
 $Comp
-L redwood:SW_PUSH SW1
+L hillside:SW_PUSH SW1
 U 1 1 6120A557
 P 3100 6300
@@
 	6300 6200 6600 6200
 $Comp
-L redwood:Mount_Trackball H2
+L hillside:Mount_Trackball H2
 U 1 1 614FB6B6
 P 9200 4800
 F 0 "H2" H 9325 4825 50  0000 L CNN
 F 1 "Trackball" H 9325 4750 50  0000 L CNN
-F 2 "redwood:Pimoroni_Trackball" H 9325 4825 50  0001 C CNN
+F 2 "hillside:Pimoroni_Trackball" H 9325 4825 50  0001 C CNN
 F 3 "" H 9325 4825 50  0001 C CNN
 	1    9200 4800
@@
 $EndComp
 $Comp
-L redwood:Mount_Tenting H1
+L hillside:Mount_Tenting H1
 U 1 1 6147F195
 P 5450 4800
 F 0 "H1" H 5600 4875 50  0000 L TNN
 F 1 "Mount_Tenting" H 5600 4725 50  0000 L BNN
-F 2 "redwood:Tenting_Puck" H 5450 4800 50  0001 C CNN
+F 2 "hillside:Tenting_Puck" H 5450 4800 50  0001 C CNN
 F 3 "" H 5450 4800 50  0001 C CNN
 	1    5450 4800
@@
 $EndComp
 $Comp
-L redwood:SW_Rotary K20
+L hillside:SW_Rotary K20
 U 1 1 6150C245
 P 2650 3900
 F 0 "K20" H 2900 4000 50  0000 L CNN
 F 1 "SW_Rotary" H 2675 3650 50  0001 C CNN
-F 2 "redwood:pg1350-DR_rotary" H 2575 4150 50  0001 C CNN
+F 2 "hillside:pg1350-DR_rotary" H 2575 4150 50  0001 C CNN
 F 3 "" H 2575 4150 50  0001 C CNN
 	1    2650 3900
@@
 Connection ~ 2150 7750
 $Comp
-L redwood:SW_Key K1
+L hillside:SW_Key K1
 U 1 1 617CBCE8
 P 950 1500
 F 0 "K1" H 950 1800 50  0000 C CNN
 F 1 "SW_Key" H 950 1700 50  0000 C CNN
-F 2 "redwood:pg1350-R" H 950 1500 50  0001 C CNN
+F 2 "hillside:pg1350-R" H 950 1500 50  0001 C CNN
 F 3 "" H 950 1500 50  0000 C CNN
 	1    950  1500
@@
 $EndComp
 $Comp
-L redwood:SW_Key K2
+L hillside:SW_Key K2
 U 1 1 617D0821
 P 1650 1500
 F 0 "K2" H 1650 1800 50  0000 C CNN
 F 1 "SW_Key" H 1650 1700 50  0000 C CNN
-F 2 "redwood:pg1350-R" H 1650 1500 50  0001 C CNN
+F 2 "hillside:pg1350-R" H 1650 1500 50  0001 C CNN
 F 3 "" H 1650 1500 50  0000 C CNN
 	1    1650 1500
@@
 $EndComp
 $Comp
-L redwood:SW_Key K3
+L hillside:SW_Key K3
 U 1 1 6183EDFD
 P 2750 1500
 F 0 "K3" H 2750 1800 50  0000 C CNN
 F 1 "SW_Key" H 2750 1700 50  0000 C CNN
-F 2 "redwood:pg1350-R" H 2750 1500 50  0001 C CNN
+F 2 "hillside:pg1350-R" H 2750 1500 50  0001 C CNN
 F 3 "" H 2750 1500 50  0000 C CNN
 	1    2750 1500
@@
 $EndComp
 $Comp
-L redwood:SW_Key K4
+L hillside:SW_Key K4
 U 1 1 6183EE07
 P 3450 1500
 F 0 "K4" H 3450 1800 50  0000 C CNN
 F 1 "SW_Key" H 3450 1700 50  0000 C CNN
-F 2 "redwood:pg1350-R" H 3450 1500 50  0001 C CNN
+F 2 "hillside:pg1350-R" H 3450 1500 50  0001 C CNN
 F 3 "" H 3450 1500 50  0000 C CNN
 	1    3450 1500
@@
 $EndComp
 $Comp
-L redwood:SW_Key K7
+L hillside:SW_Key K7
 U 1 1 6185890A
 P 950 2050
 F 0 "K7" H 950 2350 50  0000 C CNN
 F 1 "SW_Key" H 950 2250 50  0000 C CNN
-F 2 "redwood:pg1350-R" H 950 2050 50  0001 C CNN
+F 2 "hillside:pg1350-R" H 950 2050 50  0001 C CNN
 F 3 "" H 950 2050 50  0000 C CNN
 	1    950  2050
@@
 $EndComp
 $Comp
-L redwood:SW_Key K8
+L hillside:SW_Key K8
 U 1 1 61858914
 P 1650 2050
 F 0 "K8" H 1650 2350 50  0000 C CNN
 F 1 "SW_Key" H 1650 2250 50  0000 C CNN
-F 2 "redwood:pg1350-R" H 1650 2050 50  0001 C CNN
+F 2 "hillside:pg1350-R" H 1650 2050 50  0001 C CNN
 F 3 "" H 1650 2050 50  0000 C CNN
 	1    1650 2050
@@
 $EndComp
 $Comp
-L redwood:SW_Key K13
+L hillside:SW_Key K13
 U 1 1 616DA088
 P 950 2600
 F 0 "K13" H 950 2900 50  0000 C CNN
 F 1 "SW_Key" H 950 2800 50  0000 C CNN
-F 2 "redwood:pg1350-R" H 950 2600 50  0001 C CNN
+F 2 "hillside:pg1350-R" H 950 2600 50  0001 C CNN
 F 3 "" H 950 2600 50  0000 C CNN
 	1    950  2600
@@
 $EndComp
 $Comp
-L redwood:SW_Key K14
+L hillside:SW_Key K14
 U 1 1 616DA092
 P 1650 2600
 F 0 "K14" H 1650 2900 50  0000 C CNN
 F 1 "SW_Key" H 1650 2800 50  0000 C CNN
-F 2 "redwood:pg1350-R" H 1650 2600 50  0001 C CNN
+F 2 "hillside:pg1350-R" H 1650 2600 50  0001 C CNN
 F 3 "" H 1650 2600 50  0000 C CNN
 	1    1650 2600
@@
 $EndComp
 $Comp
-L redwood:SW_Key K9
+L hillside:SW_Key K9
 U 1 1 61738D17
 P 2750 2050
 F 0 "K9" H 2750 2350 50  0000 C CNN
 F 1 "SW_Key" H 2750 2250 50  0000 C CNN
-F 2 "redwood:pg1350-R" H 2750 2050 50  0001 C CNN
+F 2 "hillside:pg1350-R" H 2750 2050 50  0001 C CNN
 F 3 "" H 2750 2050 50  0000 C CNN
 	1    2750 2050
@@
 $EndComp
 $Comp
-L redwood:SW_Key K10
+L hillside:SW_Key K10
 U 1 1 61738D21
 P 3450 2050
 F 0 "K10" H 3450 2350 50  0000 C CNN
 F 1 "SW_Key" H 3450 2250 50  0000 C CNN
-F 2 "redwood:pg1350-R" H 3450 2050 50  0001 C CNN
+F 2 "hillside:pg1350-R" H 3450 2050 50  0001 C CNN
 F 3 "" H 3450 2050 50  0000 C CNN
 	1    3450 2050
@@
 $EndComp
 $Comp
-L redwood:SW_Key K15
+L hillside:SW_Key K15
 U 1 1 617598FA
 P 2750 2600
 F 0 "K15" H 2750 2900 50  0000 C CNN
 F 1 "SW_Key" H 2750 2800 50  0000 C CNN
-F 2 "redwood:pg1350-R" H 2750 2600 50  0001 C CNN
+F 2 "hillside:pg1350-R" H 2750 2600 50  0001 C CNN
 F 3 "" H 2750 2600 50  0000 C CNN
 	1    2750 2600
@@
 $EndComp
 $Comp
-L redwood:SW_Key K16
+L hillside:SW_Key K16
 U 1 1 61759904
 P 3450 2600
 F 0 "K16" H 3450 2900 50  0000 C CNN
 F 1 "SW_Key" H 3450 2800 50  0000 C CNN
-F 2 "redwood:pg1350-R" H 3450 2600 50  0001 C CNN
+F 2 "hillside:pg1350-R" H 3450 2600 50  0001 C CNN
 F 3 "" H 3450 2600 50  0000 C CNN
 	1    3450 2600
@@
 $EndComp
 $Comp
-L redwood:SW_Key K5
+L hillside:SW_Key K5
 U 1 1 617E537C
 P 4550 1500
 F 0 "K5" H 4550 1800 50  0000 C CNN
 F 1 "SW_Key" H 4550 1700 50  0000 C CNN
-F 2 "redwood:pg1350-R" H 4550 1500 50  0001 C CNN
+F 2 "hillside:pg1350-R" H 4550 1500 50  0001 C CNN
 F 3 "" H 4550 1500 50  0000 C CNN
 	1    4550 1500
@@
 $EndComp
 $Comp
-L redwood:SW_Key K6
+L hillside:SW_Key K6
 U 1 1 617E5386
 P 5250 1500
 F 0 "K6" H 5250 1800 50  0000 C CNN
 F 1 "SW_Key" H 5250 1700 50  0000 C CNN
-F 2 "redwood:pg1350-R" H 5250 1500 50  0001 C CNN
+F 2 "hillside:pg1350-R" H 5250 1500 50  0001 C CNN
 F 3 "" H 5250 1500 50  0000 C CNN
 	1    5250 1500
@@
 $EndComp
 $Comp
-L redwood:SW_Key K11
+L hillside:SW_Key K11
 U 1 1 617E53A4
 P 4550 2050
 F 0 "K11" H 4550 2350 50  0000 C CNN
 F 1 "SW_Key" H 4550 2250 50  0000 C CNN
-F 2 "redwood:pg1350-R" H 4550 2050 50  0001 C CNN
+F 2 "hillside:pg1350-R" H 4550 2050 50  0001 C CNN
 F 3 "" H 4550 2050 50  0000 C CNN
 	1    4550 2050
@@
 $EndComp
 $Comp
-L redwood:SW_Key K12
+L hillside:SW_Key K12
 U 1 1 617E53AE
 P 5250 2050
 F 0 "K12" H 5250 2350 50  0000 C CNN
 F 1 "SW_Key" H 5250 2250 50  0000 C CNN
-F 2 "redwood:pg1350-R" H 5250 2050 50  0001 C CNN
+F 2 "hillside:pg1350-R" H 5250 2050 50  0001 C CNN
 F 3 "" H 5250 2050 50  0000 C CNN
 	1    5250 2050
@@
 $EndComp
 $Comp
-L redwood:SW_Key K17
+L hillside:SW_Key K17
 U 1 1 617E53C9
 P 4550 2600
 F 0 "K17" H 4550 2900 50  0000 C CNN
 F 1 "SW_Key" H 4550 2800 50  0000 C CNN
-F 2 "redwood:pg1350-R" H 4550 2600 50  0001 C CNN
+F 2 "hillside:pg1350-R" H 4550 2600 50  0001 C CNN
 F 3 "" H 4550 2600 50  0000 C CNN
 	1    4550 2600
@@
 $EndComp
 $Comp
-L redwood:SW_Key K18
+L hillside:SW_Key K18
 U 1 1 617E53D3
 P 5250 2600
 F 0 "K18" H 5250 2900 50  0000 C CNN
 F 1 "SW_Key" H 5250 2800 50  0000 C CNN
-F 2 "redwood:pg1350-R" H 5250 2600 50  0001 C CNN
+F 2 "hillside:pg1350-R" H 5250 2600 50  0001 C CNN
 F 3 "" H 5250 2600 50  0000 C CNN
 	1    5250 2600
@@
 Connection ~ 650  2600
 $Comp
-L redwood:SW_Key K21
+L hillside:SW_Key K21
 U 1 1 619671D4
 P 3500 3600
 F 0 "K21" H 3500 3900 50  0000 C CNN
 F 1 "SW_Key" H 3500 3800 50  0000 C CNN
-F 2 "redwood:pg1350-R" H 3500 3600 50  0001 C CNN
+F 2 "hillside:pg1350-R" H 3500 3600 50  0001 C CNN
 F 3 "" H 3500 3600 50  0000 C CNN
 	1    3500 3600
@@
 $EndComp
 $Comp
-L redwood:SW_Key K22
+L hillside:SW_Key K22
 U 1 1 619CA548
 P 4600 3600
 F 0 "K22" H 4600 3900 50  0000 C CNN
 F 1 "SW_Key" H 4600 3800 50  0000 C CNN
-F 2 "redwood:pg1350-R" H 4600 3600 50  0001 C CNN
+F 2 "hillside:pg1350-R" H 4600 3600 50  0001 C CNN
 F 3 "" H 4600 3600 50  0000 C CNN
 	1    4600 3600
@@
 $EndComp
 $Comp
-L redwood:SW_Key K23
+L hillside:SW_Key K23
 U 1 1 619CA552
 P 5300 3600
 F 0 "K23" H 5300 3900 50  0000 C CNN
 F 1 "SW_Key" H 5300 3800 50  0000 C CNN
-F 2 "redwood:pg1350-R" H 5300 3600 50  0001 C CNN
+F 2 "hillside:pg1350-R" H 5300 3600 50  0001 C CNN
 F 3 "" H 5300 3600 50  0000 C CNN
 	1    5300 3600
@@
 $EndComp
 $Comp
-L redwood:SW_Key K24
+L hillside:SW_Key K24
 U 1 1 616F3997
 P 6400 3600
 F 0 "K24" H 6400 3900 50  0000 C CNN
 F 1 "SW_Key" H 6400 3800 50  0000 C CNN
-F 2 "redwood:pg1350-R" H 6400 3600 50  0001 C CNN
+F 2 "hillside:pg1350-R" H 6400 3600 50  0001 C CNN
 F 3 "" H 6400 3600 50  0000 C CNN
 	1    6400 3600
@@
 $EndComp
 $Comp
-L redwood:SW_Key K19
+L hillside:SW_Key K19
 U 1 1 616F39A1
 P 6050 2950
 F 0 "K19" H 6050 3250 50  0000 C CNN
 F 1 "SW_Key" H 6050 3150 50  0000 C CNN
-F 2 "redwood:pg1350-R" H 6050 2950 50  0001 C CNN
+F 2 "hillside:pg1350-R" H 6050 2950 50  0001 C CNN
 F 3 "" H 6050 2950 50  0000 C CNN
 	1    6050 2950
@@
 NoConn ~ 8650 1150
 $Comp
-L redwood:Scene H3
+L hillside:Scene H3
 U 1 1 62029C5C
 P 850 7050
 F 0 "H3" H 1100 7200 50  0000 L CNN
 F 1 "Scene" H 1100 7100 50  0000 L CNN
-F 2 "redwood:Hillside_Scene" H 850 6800 50  0001 C CNN
+F 2 "hillside:Hillside_Scene" H 850 6800 50  0001 C CNN
 F 3 "" H 850 6800 50  0001 C CNN
 	1    850  7050

Commit message: TRRS order has no-connect, cleanup matrix layout
Parts:
- removed D10, D11, D12, D13, D14, D15, D16, D17, D18, D7, D8, D9: BAV70, ki_syms:SOT-23, symbol ki_syms:BAV70
- added D10, D11, D12, D13, D14, D15, D16, D17, D18, D7, D8, D9: BAV70, ki_syms:SOT-23, symbol ki_syms:BAV70_Small
- added V20, V21, V22: Via, ki_syms:VIA-0.8mm, symbol ki_syms:Via
- H4, H5, H8, H9: footprint ki_mount_hole:MountingHole_2.2mm_M2_Pad -> ki_syms:MountingHole_2.2mm_M2_Pad
- H6, H7: footprint ki_mount_hole:MountingHole_2.2mm_M2 -> ki_syms:MountingHole_2.2mm_M2
- J3: value Batt_Pos -> Bat_Pos
- J4: value Batt_GND -> Bat_GND
- JP1: value SolderJumper_2_Bridged -> SolderJumper
Connections:
- wire segments 141 -> 156
- no-connect marks 4 -> 5
Other:
- moved on the sheet: C1, D1, D2, D3, D4, D5, H1, H2, H4, H5, H6, H7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

Commit message: Sym/Footprint: rename logo, cleanups
- remove unused choc-diode sym
Parts:
- H3: value Scene -> Logo; footprint hillside:Hillside_Scene -> hillside:Hillside_Logo; symbol hillside:Scene -> hillside:Logo
Changed lines of the file:
@@
 NoConn ~ 9100 1650
 $Comp
-L hillside:Scene H3
+L hillside:Logo H3
 U 1 1 62029C5C
 P 850 7050
 F 0 "H3" H 1100 7200 50  0000 L CNN
-F 1 "Scene" H 1100 7100 50  0000 L CNN
-F 2 "hillside:Hillside_Scene" H 850 6800 50  0001 C CNN
+F 1 "Logo" H 1100 7100 50  0000 L CNN
+F 2 "hillside:Hillside_Logo" H 850 6800 50  0001 C CNN
 F 3 "" H 850 6800 50  0001 C CNN
 	1    850  7050

Commit message: Common symbols/footprints used in hillside_basic
Parts:
- C1: footprint ki_syms:C_0805_2012Metric -> hillside_basic:C_0805_2012Metric; symbol ki_syms:C -> hillside_basic:C
- D1, D2, D3, D4, D5: footprint ki_syms:SK6812-MINI-E -> hillside_basic:SK6812-MINI-E; symbol ki_syms:SK6812-MINI-E -> hillside_basic:SK6812-MINI-E
- D10, D11, D12, D13, D14, D15, D16, D17, D18, D7, D8, D9: footprint ki_syms:SOT-23 -> hillside_basic:SOT-23; symbol ki_syms:BAV70_Small -> hillside_basic:BAV70_Small
- H4, H5, H8, H9: footprint ki_syms:MountingHole_2.2mm_M2_Pad -> hillside_basic:MountingHole_2.2mm_M2_Pad; symbol ki_mech:MountingHole -> hillside_basic:MountingHole
- H6, H7: footprint ki_syms:MountingHole_2.2mm_M2 -> hillside_basic:MountingHole_2.2mm_M2; symbol ki_mech:MountingHole -> hillside_basic:MountingHole
- J1: symbol ki_syms:Conn_01x05-Connector_Generic -> hillside_basic:Conn_01x05-Connector_Generic
- J3, J4: footprint ki_syms:1pin_conn -> hillside_basic:1pin_conn; symbol ki_conn_generic:Conn_01x01 -> hillside_basic:Conn_01x01
- JP1: footprint ki_syms:SolderJumper-2_P1.3mm_Bridged_RoundedPad1.0x1.5mm -> hillside_basic:SolderJumper-2_P1.3mm_Bridged_RoundedPad1.0x1.5mm; symbol ki_jumper:SolderJumper_2_Bridged -> hillside_basic:SolderJumper_2_Bridged
- R1, R2: footprint ki_syms:R_0805_2012Metric -> hillside_basic:R_0805_2012Metric; symbol ki_syms:R -> hillside_basic:R
- SW1: footprint ki_syms:SW_SPST_SKQG_WithStem -> hillside_basic:SW_SPST_SKQG_WithStem
- SW2: footprint ki_syms:SW_SPDT_JS202011AQN -> hillside_basic:SW_SPDT_JS202011AQN; symbol ki_switch:SW_SPDT -> hillside_basic:SW_SPDT
- V1, V10, V11, V12, V13, V14, V15, V16, V17, V18, V19, V2, V20, V21, V22, V3, V4, V5, V6, V7, V8, V9: footprint ki_syms:VIA-0.8mm -> hillside_basic:VIA-0.8mm; symbol ki_syms:Via -> hillside_basic:Via

Commit message: - cleanup schema sheet
Parts:
- V1: value V -> Via
Other:
- note added: "KiCad"
- moved on the sheet: C1, D1, D10, D11, D12, D13, D14, D15, D16, D17, D18, D2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
