File: hillside46/hillside46.kicad_pcb (KiCad board)
At the start: 2 copper layers, 142.5 x 99.9 mm, 86 parts, among them J1 Haptic, J2 TRRS, J3 Bat_Pos, J4 Bat_Neg, J5 Bat_Pos, J6 Bat_Neg, K1 SW_Key, K10 SW_Key, K11 SW_Key, K12 SW_Key, K13 SW_Key, K14 SW_Key, K15 SW_Key, K16 SW_Key, K17 SW_Key, K18 SW_Key, K19 SW_Rotary, K2 SW_Key, K20 SW_Rotary, K21 SW_Key, K22 SW_Key, K23 SW_Key, K3 SW_Key, K4 SW_Key, K5 SW_Key, K6 SW_Key, K7 SW_Key, K8 SW_Key, K9 SW_Key, SW1 SKQGAFE010, SW2 SW_Power, U1 ProMicro_r, U2 SRV05-4

Commit message: 46: Flip resistor to test back positioning
Parts:
- R2: moved to B.Cu
Changed lines of the file:
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@@
       ))
-  )
-  (footprint "hillside_basic:R_0805_2012Metric" (layer "F.Cu")
-    (at 209.745771 82.312259 90)
-    (descr "Resistor SMD 0805 (2012 Metric), square (rectangular) end terminal, IPC_7351 nominal, (Body size source: IPC-SM-782 page 72, https://www.pcb-3d.com/wordpress/wp-content/uploads/ipc-sm-782a_amendment_1_and_2.pdf), generated with kicad-footprint-generator")
-    (tags "resistor")
-    (property "Config" "Optional")
-    (property "JLC Type" "Basic")
-    (property "LCSC" "C17673")
-    (property "Price" ".002 @20+")
-    (property "Sheetfile" "hillside46.kicad_sch")
-    (property "Sheetname" "")
-    (attr smd)
-    (fp_text reference "R2" (at 0.045142 1.637337 90) (layer "F.Fab")
-      (effects (font (size 1 1) (thickness 0.153)))
-    )
-    (fp_text value "4.7k" (at 1.420142 -1.212663 90) (layer "F.SilkS")
-      (effects (font (size 0.9 0.6) (thickness 0.15)))
-    )
-    (fp_text user "${REFERENCE}" (at 0 0 90) (layer "F.Fab")
-      (effects (font (size 0.5 0.5) (thickness 0.08)))
-    )
-    (fp_line (start -0.227064 0.735) (end 0.227064 0.735) (layer "F.SilkS") (width 0.12))
-    (fp_line (start -0.227064 -0.735) (end 0.227064 -0.735) (layer "F.SilkS") (width 0.12))
-    (fp_line (start 1.68 -0.95) (end 1.68 0.95) (layer "F.CrtYd") (width 0.05))
-    (fp_line (start 1.68 0.95) (end -1.68 0.95) (layer "F.CrtYd") (width 0.05))
-    (fp_line (start -1.68 -0.95) (end 1.68 -0.95) (layer "F.CrtYd") (width 0.05))
-    (fp_line (start -1.68 0.95) (end -1.68 -0.95) (layer "F.CrtYd") (width 0.05))
-    (fp_line (start -1 0.625) (end -1 -0.625) (layer "F.Fab") (width 0.1))
-    (fp_line (start 1 -0.625) (end 1 0.625) (layer "F.Fab") (width 0.1))
-    (fp_line (start -1 -0.625) (end 1 -0.625) (layer "F.Fab") (width 0.1))
-    (fp_line (start 1 0.625) (end -1 0.625) (layer "F.Fab") (width 0.1))
-    (pad "1" smd roundrect (at -0.9125 0 90) (size 1.025 1.4) (layers "B.Cu" "B.Paste" "B.Mask") (roundrect_rratio 0.244)
-      (net 46 "VCC_ACC") (pintype "passive"))
-    (pad "1" thru_hole custom (at -2.1 0 90) (size 0.8 0.8) (drill 0.4) (layers *.Cu)
-      (net 46 "VCC_ACC") (pintype "passive") (zone_connect 0)
-      (options (clearance outline) (anchor circle))
-      (primitives
-        (gr_line (start 1.1875 0) (end 0 0) (width 0.254))
-      ))
-    (pad "1" smd roundrect (at -0.9125 0 90) (size 1.025 1.4) (layers "F.Cu" "F.Paste" "F.Mask") (roundrect_rratio 0.244)
-      (net 46 "VCC_ACC") (pintype "passive"))
-    (pad "2" smd roundrect (at 0.9125 0 90) (size 1.025 1.4) (layers "F.Cu" "F.Paste" "F.Mask") (roundrect_rratio 0.243902439)
-      (net 20 "SDA") (pintype "passive"))
-    (pad "2" smd roundrect (at 0.9125 0 90) (size 1.025 1.4) (layers "B.Cu" "B.Paste" "B.Mask") (roundrect_rratio 0.244)
-      (net 20 "SDA") (pintype "passive"))
-    (pad "2" thru_hole custom (at 2.1 0 90) (size 0.8 0.8) (drill 0.4) (layers *.Cu)
-      (net 20 "SDA") (pintype "passive") (zone_connect 0)
-      (options (clearance outline) (anchor circle))
-      (primitives
-        (gr_line (start -1.1875 0) (end 0 0) (width 0.254))
-      ))
-    (model "${KISYS3DMOD}/Resistor_SMD.3dshapes/R_0805_2012Metric.wrl"
-      (offset (xyz 0 0 0))
-      (scale (xyz 1 1 1))
-      (rotate (xyz 0 0 0))
-    )
   )
   (footprint "hillside:Pimoroni_Haptic" (layer "F.Cu")
@@
     (fp_circle (center 0 0) (end 3.95 0) (layer "User.2") (width 0.12) (fill none))
   )
+  (footprint "hillside_basic:R_0805_2012Metric" (layer "B.Cu")
+    (at 209.745771 82.312259 90)
+    (descr "Resistor SMD 0805 (2012 Metric), square (rectangular) end terminal, IPC_7351 nominal, (Body size source: IPC-SM-782 page 72, https://www.pcb-3d.com/wordpress/wp-content/uploads/ipc-sm-782a_amendment_1_and_2.pdf), generated with kicad-footprint-generator")
+    (tags "resistor")
+    (property "Config" "Optional")
+    (property "JLC Type" "Basic")
+    (property "LCSC" "C17673")
+    (property "Price" ".002 @20+")
+    (property "Sheetfile" "hillside46.kicad_sch")
+    (property "Sheetname" "")
+    (attr smd)
+    (fp_text reference "R2" (at 0.045142 -1.637337 90) (layer "B.Fab")
+      (effects (font (size 1 1) (thickness 0.153)) (justify mirror))
+    )
+    (fp_text value "4.7k" (at 1.420142 1.212663 90) (layer "B.SilkS")
+      (effects (font (size 0.9 0.6) (thickness 0.15)) (justify mirror))
+    )
+    (fp_text user "${REFERENCE}" (at 0 0 90) (layer "B.Fab")
+      (effects (font (size 0.5 0.5) (thickness 0.08)) (justify mirror))
+    )
+    (fp_line (start -0.227064 -0.735) (end 0.227064 -0.735) (layer "B.SilkS") (width 0.12))
+    (fp_line (start -0.227064 0.735) (end 0.227064 0.735) (layer "B.SilkS") (width 0.12))
+    (fp_line (start 1.68 0.95) (end 1.68 -0.95) (layer "B.CrtYd") (width 0.05))
+    (fp_line (start 1.68 -0.95) (end -1.68 -0.95) (layer "B.CrtYd") (width 0.05))
+    (fp_line (start -1.68 0.95) (end 1.68 0.95) (layer "B.CrtYd") (width 0.05))
+    (fp_line (start -1.68 -0.95) (end -1.68 0.95) (layer "B.CrtYd") (width 0.05))
+    (fp_line (start -1 -0.625) (end -1 0.625) (layer "B.Fab") (width 0.1))
+    (fp_line (start 1 0.625) (end 1 -0.625) (layer "B.Fab") (width 0.1))
+    (fp_line (start -1 0.625) (end 1 0.625) (layer "B.Fab") (width 0.1))
+    (fp_line (start 1 -0.625) (end -1 -0.625) (layer "B.Fab") (width 0.1))
+    (pad "1" smd roundrect (at -0.9125 0 90) (size 1.025 1.4) (layers "F.Cu" "F.Paste" "F.Mask") (roundrect_rratio 0.244)
+      (net 46 "VCC_ACC") (pintype "passive"))
+    (pad "1" thru_hole custom (at -2.1 0 90) (size 0.8 0.8) (drill 0.4) (layers *.Cu)
+      (net 46 "VCC_ACC") (pintype "passive") (zone_connect 0)
+      (options (clearance outline) (anchor circle))
+      (primitives
+        (gr_line (start 0 0) (end 1.1875 0) (width 0.254))
+      ))
+    (pad "1" smd roundrect (at -0.9125 0 90) (size 1.025 1.4) (layers "B.Cu" "B.Paste" "B.Mask") (roundrect_rratio 0.244)
+      (net 46 "VCC_ACC") (pintype "passive"))
+    (pad "2" smd roundrect (at 0.9125 0 90) (size 1.025 1.4) (layers "B.Cu" "B.Paste" "B.Mask") (roundrect_rratio 0.243902439)
+      (net 20 "SDA") (pintype "passive"))
+    (pad "2" smd roundrect (at 0.9125 0 90) (size 1.025 1.4) (layers "F.Cu" "F.Paste" "F.Mask") (roundrect_rratio 0.244)
+      (net 20 "SDA") (pintype "passive"))
+    (pad "2" thru_hole custom (at 2.1 0 90) (size 0.8 0.8) (drill 0.4) (layers *.Cu)
+      (net 20 "SDA") (pintype "passive") (zone_connect 0)
+      (options (clearance outline) (anchor circle))
+      (primitives
+        (gr_line (start 0 0) (end -1.1875 0) (width 0.254))
+      ))
+    (model "${KISYS3DMOD}/Resistor_SMD.3dshapes/R_0805_2012Metric.wrl"
+      (offset (xyz 0 0 0))
+      (scale (xyz 1 1 1))
+      (rotate (xyz 0 0 0))
+    )
+  )
   (gr_line (start 150.625769 48.792254) (end 135.885771 48.792263) (layer "Edge.Cuts") (width 0.05))
